Commit message: pushbot sim working, controllers in progress

File: examples/pushbot/urdf/pushbot.urdf (robot description, URDF)
Before this commit: robot pushbot, 3 links, 2 joints
Links:
- added link ee_slider; visual box size=0.05 0.05 0.3
- link arm: geometry collision cylinder length=1.0 radius=0.05; visual cylinder length=1.0 radius=0.05
- link base: geometry collision cylinder length=0.07 radius=0.1; visual cylinder length=0.07 radius=0.1
- link end_effector: geometry collision sphere radius=0.075; visual sphere radius=0.075
Joints:
- added joint ee_slider_joint: type fixed, parent arm, child ee_slider, origin xyz=0 0 1.0 rpy=0 0 0
- joint push_joint: origin xyz=0 0.16 0 rpy=0 0 0 -> xyz=0 0 1.0 rpy=0 0 0
